File: hw/tragic-8-ball/tragic-8-ball.kicad_sch (KiCad schematic)
At the start: 7 parts

Commit message: schematic and pinout'
Parts:
- added D2, D3, D4, D5, D6: LED, symbol Device:LED
- added DISP1: special_LCD, symbol symbols-local:special_LCD
- added H? (x4): MountingHole_Pad, symbol Mechanical:MountingHole_Pad
- added R3: 10k, symbol Device:R_US
- added R4, R5, R6, R7, R8: 1k, symbol Device:R_US
- added SW1: SW_SPST, symbol Switch:SW_SPST
- added SW2: SW_Push, symbol Switch:SW_Push
- gave numbers to parts that had none: 7
Connections:
- net +3V0: now also SW1.1 (A); no longer R1.1
- net GND: now also H?.1, H?.1, H?.1, H?.1, SW2.1
- net VDD: now also R3.1, R4.2, R5.2, R6.2, R7.2, R8.2
- net LED5: now reaches U1.10 (PA4)
- net LED5: now also D2.1 (K)
- net LED4: now reaches U1.11 (PA5)
- net LED4: now also D3.1 (K)
- net LED3: now reaches U1.12 (PA6)
- net LED3: now also D4.1 (K)
- net LED2: now reaches U1.13 (PA7)
- net LED2: now also D5.1 (K)
- net SWITCH: now reaches U1.14 (PB1)
- net SWITCH: now also R3.2, SW2.2
- net LED1: now reaches U1.17 (PA9)
- net LED1: now also D6.1 (K)
- net REF: now reaches U1.18 (PA10)
- net REF: now also DISP1.1 (REF)
- net B_CTRL: now reaches U1.6 (PA0)
- net B_CTRL: now also DISP1.2 (B)
- net H_CTRL: now reaches U1.7 (PA1)
- net H_CTRL: now also DISP1.3 (H)
- net N_CTRL: now reaches U1.8 (PA2)
- net N_CTRL: now also DISP1.4 (N)
- net P_CTRL: now reaches U1.9 (PA3)
- net P_CTRL: now also DISP1.5 (P)
- new net: D6.2 (A), R8.1
- new net: D3.2 (A), R5.1
- new net: D2.2 (A), R4.1
- new net: D4.2 (A), R6.1
- new net: R1.1, SW1.2 (B)
- new net: D5.2 (A), R7.1
Other:
- moved on the sheet: BT1, J1
